Commit message: Can now recreate any trajectory in gazebo

File: urdf/panda_camera.xacro (robot description, xacro)
@@ -89,3 +89,53 @@
     </plugin>
   </gazebo>
+<!-- ============================================ -->
+  <!-- MATÉRIAUX GAZEBO (pour les couleurs)         -->
+  <!-- ============================================ -->
+  <!-- Couleur blanche pour tous les liens du bras -->
+  <gazebo reference="$(arg arm_id)_link0">
+    <material>Gazebo/White</material>
+  </gazebo>
+  <gazebo reference="$(arg arm_id)_link1">
+    <material>Gazebo/White</material>
+  </gazebo>
+  <gazebo reference="$(arg arm_id)_link2">
+    <material>Gazebo/White</material>
+  </gazebo>
+  <gazebo reference="$(arg arm_id)_link3">
+    <material>Gazebo/White</material>
+  </gazebo>
+  <gazebo reference="$(arg arm_id)_link4">
+    <material>Gazebo/White</material>
+  </gazebo>
+  <gazebo reference="$(arg arm_id)_link5">
+    <material>Gazebo/White</material>
+  </gazebo>
+  <gazebo reference="$(arg arm_id)_link6">
+    <material>Gazebo/White</material>
+  </gazebo>
+  <gazebo reference="$(arg arm_id)_link7">
+    <material>Gazebo/White</material>
+  </gazebo>
+  <gazebo reference="$(arg arm_id)_link8">
+    <material>Gazebo/White</material>
+  </gazebo>
+  <!-- Gripper en gris foncé -->
+  <gazebo reference="$(arg arm_id)_hand">
+    <material>Gazebo/DarkGrey</material>
+  </gazebo>
+  <gazebo reference="$(arg arm_id)_leftfinger">
+    <material>Gazebo/DarkGrey</material>
+  </gazebo>
+  <gazebo reference="$(arg arm_id)_rightfinger">
+    <material>Gazebo/DarkGrey</material>
+  </gazebo>
+  <gazebo reference="$(arg arm_id)_hand">
+    <material>Gazebo/White</material>
+  </gazebo>
+  <gazebo reference="$(arg arm_id)_leftfinger">
+    <material>Gazebo/White</material>
+  </gazebo>
+  <gazebo reference="$(arg arm_id)_rightfinger">
+    <material>Gazebo/White</material>
+  </gazebo>
 </robot>

Commit message: Presque réussi le temps réel, saccade et semble ne pas avoir un bon buffer

File: urdf/panda_camera.xacro (robot description, xacro)
@@ -19,10 +19,10 @@
     <visual>
       <origin xyz="-0.033 -0.02 0.0171378" rpy="0 ${27.5 * pi / 180} 0"/>
-      <geometry><mesh filename="$(find vision_processing)/src/vision_processing/diffusion_model_train/fork.STL" scale="0.001 0.001 0.001"/></geometry>
+      <geometry><mesh filename="package://vision_processing/src/vision_processing/diffusion_model_train/fork.STL" scale="0.001 0.001 0.001"/></geometry>
     </visual>
-    <collision>
+    <!-- <collision>
       <origin xyz="-0.033 -0.02 0.0171378" rpy="0 ${27.5 * pi / 180} 0"/>
-      <geometry><mesh filename="$(find vision_processing)/src/vision_processing/diffusion_model_train/fork.STL" scale="0.001 0.001 0.001"/></geometry>
-    </collision>
+      <geometry><mesh filename="package://vision_processing/src/vision_processing/diffusion_model_train/fork.STL" scale="0.001 0.001 0.001"/></geometry>
+    </collision> -->
     <inertial> <mass value="0.1" />
       <inertia ixx="0.0001" ixy="0" ixz="0" iyy="0.0001" iyz="0" izz="0.0001" />
@@ -93,5 +93,5 @@
     <material>Gazebo/Red</material>
     <sensor type="depth" name="camera_static">
-      <update_rate>30.0</update_rate>
+      <update_rate>15.0</update_rate>
       <camera>
         <horizontal_fov>0.958</horizontal_fov>
@@ -112,9 +112,15 @@
     <material>Gazebo/Blue</material>
     <sensor type="depth" name="camera_wrist">
-      <update_rate>30.0</update_rate>
+      <update_rate>15.0</update_rate>
       <camera>
         <horizontal_fov>0.973</horizontal_fov>
-        <image><width>640</width><height>480</height><format>R8G8B8</format></image>
-        <clip><near>0.05</near><far>3.0</far></clip>
+        <image>
+            <width>640</width>
+            <height>480</height>
+            <format>R8G8B8</format>
+        </image>
+        <clip>
+            <near>0.01</near> <far>10.0</far>
+        </clip>
       </camera>
       <plugin name="wrist_camera_controller" filename="libgazebo_ros_openni_kinect.so">
@@ -125,4 +131,7 @@
         <cameraInfoTopicName>color/camera_info</cameraInfoTopicName>
         <frameName>camera_wrist_optical_frame</frameName>
+        <pointCloudCutoff>0.01</pointCloudCutoff>
+        <pointCloudCutoffMax>10.0</pointCloudCutoffMax>
+        <updateRate>15.0</updateRate>
       </plugin>
     </sensor>
