Commit message: Update

File: urdf/food.urdf (robot description, URDF)
Before this commit: robot food_cube, 1 links, 0 joints
Links:
- link base_link: geometry collision box size=0.025 0.025 0.025; visual box size=0.05 0.05 0.05

Commit message: Update

File: urdf/food.urdf (robot description, URDF)
Before this commit: robot food_cube, 1 links, 0 joints
Links:
- link base_link: geometry collision box size=0.025 0.025 0.005; visual box size=0.025 0.025 0.005

File: urdf/panda_camera.xacro (robot description, xacro)
@@ -21,8 +21,4 @@
       <geometry><mesh filename="package://vision_processing/src/vision_processing/diffusion_model_train/fork.STL" scale="0.001 0.001 0.001"/></geometry>
     </visual>
-    <!-- <collision>
-      <origin xyz="-0.033 -0.02 0.0171378" rpy="0 ${27.5 * pi / 180} 0"/>
-      <geometry><mesh filename="package://vision_processing/src/vision_processing/diffusion_model_train/fork.STL" scale="0.001 0.001 0.001"/></geometry>
-    </collision> -->
     <inertial> <mass value="0.1" />
       <inertia ixx="0.0001" ixy="0" ixz="0" iyy="0.0001" iyz="0" izz="0.0001" />
@@ -34,4 +30,13 @@
     <child link="fork_tip"/>
   </joint>
+  <!-- ============================================================
+       CONTAINER (Bowl/Plate) — for SafeFlow SDF integration
+       ============================================================
+       Adjust xyz and rpy to match where you place the real container.
+       This publishes "container_link" in TF so the inference node
+       can look it up automatically.
+       ============================================================ -->
+  <xacro:include filename="$(find vision_processing)/urdf/container.xacro"/>
+  <xacro:container xyz="0.5 0.0 0.0" rpy="0 0 0"/>
   <xacro:macro name="create_transmission" params="joint_name">
     <transmission name="${joint_name}_tran">
@@ -57,5 +62,4 @@
     <child link="camera_static_link" />
     <origin xyz="1.1593 1.2922 1.1910" rpy="0.0000 0.6013 -2.3020" />
-    <!-- <origin xyz="1.1593 1.2922 1.1910" rpy="-1.967 0.009 2.559" /> -->
   </joint>
   <link name="camera_static_link">

Commit message: It worked for the first time yahoo!

File: urdf/food.urdf (robot description, URDF)
Before this commit: robot food_cube, 1 links, 0 joints
Links:
- link base_link: geometry collision box size=0.025 0.025 0.025; visual box size=0.025 0.025 0.025

File: urdf/panda_camera.xacro (robot description, xacro)
@@ -1,13 +1,11 @@
 <?xml version="1.0"?>
 <robot xmlns:xacro="http://www.ros.org/wiki/xacro" name="panda">
-  <xacro:include filename="$(find franka_description)/robots/common/franka_arm.xacro"/>
-  <xacro:include filename="$(find franka_description)/robots/common/franka_hand.xacro"/>
+  <xacro:include filename="$(find franka_description)/robots/common/franka_robot.xacro"/>
   <xacro:arg name="arm_id" default="panda" />
-  <link name="world" />
-  <xacro:franka_arm arm_id="$(arg arm_id)" connected_to="world" xyz="0 0 0"
-                    safety_distance="0.03" gazebo="true"
-                    joint_limits="${xacro.load_yaml('$(find franka_description)/robots/panda/joint_limits.yaml')}"/>
-  <xacro:franka_hand arm_id="$(arg arm_id)" rpy="0 0 ${-pi/4}"
-                    connected_to="$(arg arm_id)_link8" safety_distance="0.03" gazebo="true"/>
+  <xacro:franka_robot arm_id="$(arg arm_id)"
+                       joint_limits="${xacro.load_yaml('$(find franka_description)/robots/panda/joint_limits.yaml')}"
+                       parent="world"
+                       hand="true"
+                       gazebo="true"/>
   <link name="panda_TCP"/>
   <joint name="panda_TCP_joint" type="fixed">
@@ -19,5 +17,5 @@
     <visual>
       <origin xyz="-0.033 -0.02 0.0171378" rpy="0 ${27.5 * pi / 180} 0"/>
-      <geometry><mesh filename="package://vision_processing/src/vision_processing/diffusion_model_train/fork.STL" scale="0.001 0.001 0.001"/></geometry>
+      <geometry><mesh filename="package://vision_processing/src/vision_processing/diffusion_model_train/fork_tip.stl" scale="0.001 0.001 0.001"/></geometry>
     </visual>
     <inertial> <mass value="0.1" />
@@ -30,23 +28,14 @@
     <child link="fork_tip"/>
   </joint>
-  <xacro:macro name="create_transmission" params="joint_name">
-    <transmission name="${joint_name}_tran">
-      <type>transmission_interface/SimpleTransmission</type>
-      <joint name="${joint_name}">
-        <hardwareInterface>hardware_interface/PositionJointInterface</hardwareInterface>
-      </joint>
-      <actuator name="${joint_name}_motor">
-        <hardwareInterface>hardware_interface/PositionJointInterface</hardwareInterface>
-        <mechanicalReduction>1</mechanicalReduction>
-      </actuator>
-    </transmission>
-  </xacro:macro>
-  <xacro:create_transmission joint_name="$(arg arm_id)_joint1"/>
-  <xacro:create_transmission joint_name="$(arg arm_id)_joint2"/>
-  <xacro:create_transmission joint_name="$(arg arm_id)_joint3"/>
-  <xacro:create_transmission joint_name="$(arg arm_id)_joint4"/>
-  <xacro:create_transmission joint_name="$(arg arm_id)_joint5"/>
-  <xacro:create_transmission joint_name="$(arg arm_id)_joint6"/>
-  <xacro:create_transmission joint_name="$(arg arm_id)_joint7"/>
+  <!-- Physical tine tip: centroid of fork tine endpoints in fork_tip frame.
+       Computed from fork_tip.stl bounding box (top-1% Z vertices, scale 0.001):
+         STL tip ~ [30.5, 19.8, 180.0] mm → R_y(27.5°) × tip_m + visual_offset
+       Result: [0.0771, -0.0002, 0.1627] in fork_tip frame. -->
+  <link name="fork_tine_tip"/>
+  <joint name="fork_tine_tip_joint" type="fixed">
+    <origin xyz="0.0771 -0.0002 0.1627" rpy="0 0 0"/>
+    <parent link="fork_tip"/>
+    <child link="fork_tine_tip"/>
+  </joint>
   <joint name="camera_static_joint" type="fixed">
     <parent link="world" />
@@ -132,9 +121,3 @@
     </sensor>
   </gazebo>
-  <gazebo>
-    <plugin name="gazebo_ros_control" filename="libgazebo_ros_control.so">
-      <robotNamespace>/</robotNamespace>
-      <robotSimType>gazebo_ros_control/DefaultRobotHWSim</robotSimType>
-    </plugin>
-  </gazebo>
 </robot>

Commit message: Added grasp and now is smooth

File: urdf/food.urdf (robot description, URDF)
Before this commit: robot food_cube, 1 links, 0 joints
Links:
- link base_link: geometry collision box size=0.03 0.03 0.03; visual box size=0.025 0.025 0.025

File: urdf/panda_camera.xacro (robot description, xacro)
@@ -28,4 +28,11 @@
     <child link="fork_tip"/>
   </joint>
+  <!-- Keep fork_tip as a standalone Gazebo link (do not lump it into its
+       fixed-joint parent) so gazebo_ros_link_attacher can weld the food cube
+       to it. The fixed joint stays a rigid (zero-DOF) weld to panda_TCP. -->
+  <gazebo reference="fork_tip_joint">
+    <disableFixedJointLumping>true</disableFixedJointLumping>
+    <preserveFixedJoint>true</preserveFixedJoint>
+  </gazebo>
   <!-- Physical tine tip: centroid of fork tine endpoints in fork_tip frame.
        Computed from fork_tip.stl bounding box (top-1% Z vertices, scale 0.001):
