Commit message: Ajout des submodules

File: urdf/container.xacro (robot description, xacro)
@@ -1,58 +1,40 @@
 <?xml version="1.0"?>
-<!--
-  Container (Bowl/Plate) URDF — for SafeFlow SDF integration
-  ============================================================
-  The mesh 03_surface_aligned.obj is PCA-aligned, meaning its vertices
-  are already expressed in the container's local coordinate frame — the
-  SAME frame where the SDF was computed. No visual origin offset is needed.
-  The joint origin (xyz, rpy) defines T_world_container directly.
-  This frame is published in TF as "container_link", so the inference
-  node can look it up instead of hardcoding ~container_pose.
-  Usage in panda_camera.xacro:
-  ─────────────────────────────
-    <xacro:include filename="$(find vision_processing)/urdf/container.xacro"/>
-    <xacro:container xyz="0.5 0.3 0.0" rpy="0 0 0"/>
-  The xyz/rpy should match where you place the real bowl in the world.
--->
 <robot xmlns:xacro="http://www.ros.org/wiki/xacro" name="container">
-  <xacro:macro name="container" params="xyz:='0.5 0.0 0.0' rpy:='0 0 0'">
-    <!-- Container visual + collision link -->
-    <link name="container_link">
-      <visual>
-        <origin xyz="0 0 0" rpy="0 0 0"/>
-        <geometry>
-          <mesh filename="package://vision_processing/src/vision_processing/SDF/03_surface_aligned.obj"/>
-        </geometry>
-        <material name="container_material">
-          <color rgba="0.85 0.75 0.65 0.6"/>
-        </material>
-      </visual>
-      <!-- Collision is optional here: the fork_tip has no collision geometry,
-           so Gazebo won't detect fork-bowl contact regardless.
-           The real safety comes from the SDF + FMBF in the inference node,
-           which steers trajectories AROUND the bowl at the planning level.
-           We keep collision so the panda arm links can't clip through. -->
-      <collision>
-        <origin xyz="0 0 0" rpy="0 0 0"/>
-        <geometry>
-          <mesh filename="package://vision_processing/src/vision_processing/SDF/03_surface_aligned.obj"/>
-        </geometry>
-      </collision>
-      <inertial>
-        <mass value="0.3"/>
-        <inertia ixx="1e-3" ixy="0" ixz="0" iyy="1e-3" iyz="0" izz="1e-3"/>
-      </inertial>
-    </link>
-    <!-- Fixed joint: world → container -->
-    <joint name="container_joint" type="fixed">
-      <parent link="world"/>
-      <child link="container_link"/>
-      <origin xyz="${xyz}" rpy="${rpy}"/>
-    </joint>
-    <!-- Gazebo appearance -->
-    <gazebo reference="container_link">
-      <material>Gazebo/Wood</material>
-      <static>true</static>
-    </gazebo>
-  </xacro:macro>
+  <xacro:property name="mesh_scale" value="0.025 0.025 0.025"/>
+  <link name="container_link">
+    <visual>
+      <origin xyz="0 0 0" rpy="0 0 0"/>
+      <geometry>
+        <mesh filename="package://vision_processing/urdf/basic-bowl/source/Basic Bowl/Bowl.obj" scale="${mesh_scale}"/>
+      </geometry>
+      <material name="container_material">
+        <color rgba="1.0 1.0 1.0 1.0"/>
+      </material>
+    </visual>
+    <collision>
+      <origin xyz="0 0 0" rpy="0 0 0"/>
+      <geometry>
+        <mesh filename="package://vision_processing/urdf/basic-bowl/source/Basic Bowl/Bowl.obj" scale="${mesh_scale}"/>
+      </geometry>
+    </collision>
+    <inertial>
+      <mass value="0.3"/>
+      <inertia ixx="1e-3" ixy="0" ixz="0" iyy="1e-3" iyz="0" izz="1e-3"/>
+    </inertial>
+  </link>
+  <gazebo reference="container_link">
+    <material>Gazebo/White</material>
+  </gazebo>
+  <gazebo>
+    <plugin name="p3d_base_controller" filename="libgazebo_ros_p3d.so">
+      <alwaysOn>true</alwaysOn>
+      <updateRate>50.0</updateRate>
+      <bodyName>container_link</bodyName>
+      <topicName>container_pose</topicName>
+      <gaussianNoise>0.0</gaussianNoise>
+      <frameName>world</frameName>
+      <xyzOffsets>0 0 0</xyzOffsets>
+      <rpyOffsets>0 0 0</rpyOffsets>
+    </plugin>
+  </gazebo>
 </robot>

File: urdf/food.urdf (robot description, URDF)
Before this commit: robot food_cube, 1 links, 0 joints
Links:
- link base_link: geometry collision box size=0.025 0.025 0.005; visual box size=0.025 0.025 0.025

File: urdf/panda_camera.xacro (robot description, xacro)
@@ -9,5 +9,5 @@
                     joint_limits="${xacro.load_yaml('$(find franka_description)/robots/panda/joint_limits.yaml')}"/>
   <xacro:franka_hand arm_id="$(arg arm_id)" rpy="0 0 ${-pi/4}"
-                     connected_to="$(arg arm_id)_link8" safety_distance="0.03" gazebo="true"/>
+                    connected_to="$(arg arm_id)_link8" safety_distance="0.03" gazebo="true"/>
   <link name="panda_TCP"/>
   <joint name="panda_TCP_joint" type="fixed">
@@ -30,13 +30,4 @@
     <child link="fork_tip"/>
   </joint>
-  <!-- ============================================================
-       CONTAINER (Bowl/Plate) — for SafeFlow SDF integration
-       ============================================================
-       Adjust xyz and rpy to match where you place the real container.
-       This publishes "container_link" in TF so the inference node
-       can look it up automatically.
-       ============================================================ -->
-  <xacro:include filename="$(find vision_processing)/urdf/container.xacro"/>
-  <xacro:container xyz="0.5 0.0 0.0" rpy="0 0 0"/>
   <xacro:macro name="create_transmission" params="joint_name">
     <transmission name="${joint_name}_tran">
@@ -97,5 +88,5 @@
     <material>Gazebo/Red</material>
     <sensor type="depth" name="camera_static">
-      <update_rate>6.0</update_rate>
+      <update_rate>12.0</update_rate>
       <camera>
         <horizontal_fov>0.958</horizontal_fov>
@@ -116,5 +107,5 @@
     <material>Gazebo/Blue</material>
     <sensor type="depth" name="camera_wrist">
-      <update_rate>6.0</update_rate>
+      <update_rate>12.0</update_rate>
       <camera>
         <horizontal_fov>0.973</horizontal_fov>
@@ -137,5 +128,5 @@
         <pointCloudCutoff>0.01</pointCloudCutoff>
         <pointCloudCutoffMax>10.0</pointCloudCutoffMax>
-        <updateRate>6.0</updateRate>
+        <updateRate>12.0</updateRate>
       </plugin>
     </sensor>

File: urdf/panda_fork.urdf (robot description, URDF)
Before this commit: robot panda, 29 links, 28 joints
Joints:
- removed joint panda_joint1
- removed joint panda_joint2
- removed joint panda_joint3
- removed joint panda_joint4
- removed joint panda_joint5
- removed joint panda_joint6
- removed joint panda_joint7
- removed joint panda_joint8
- removed joint panda_joint_world
- added joint joint1: type revolute, parent panda_link0, child panda_link1, origin xyz=0 0 0.333 rpy=0 0 0, axis 0 0 1, limit lower=-2.8973 upper=2.8973 effort=87.0 velocity=2.175
- added joint joint2: type revolute, parent panda_link1, child panda_link2, origin xyz=0 0 0 rpy=-1.5707963267948966 0 0, axis 0 0 1, limit lower=-1.7628 upper=1.7628 effort=87.0 velocity=2.175
- added joint joint3: type revolute, parent panda_link2, child panda_link3, origin xyz=0 -0.316 0 rpy=1.5707963267948966 0 0, axis 0 0 1, limit lower=-2.8973 upper=2.8973 effort=87.0 velocity=2.175
- added joint joint4: type revolute, parent panda_link3, child panda_link4, origin xyz=0.0825 0 0 rpy=1.5707963267948966 0 0, axis 0 0 1, limit lower=-3.0718 upper=-0.0698 effort=87.0 velocity=2.175
- added joint joint5: type revolute, parent panda_link4, child panda_link5, origin xyz=-0.0825 0.384 0 rpy=-1.5707963267948966 0 0, axis 0 0 1, limit lower=-2.8973 upper=2.8973 effort=12.0 velocity=2.61
- added joint joint6: type revolute, parent panda_link5, child panda_link6, origin xyz=0 0 0 rpy=1.5707963267948966 0 0, axis 0 0 1, limit lower=-0.0175 upper=3.7525 effort=12.0 velocity=2.61
- added joint joint7: type revolute, parent panda_link6, child panda_link7, origin xyz=0.088 0 0 rpy=1.5707963267948966 0 0, axis 0 0 1, limit lower=-2.8973 upper=2.8973 effort=12.0 velocity=2.61
- added joint joint8: type fixed, parent panda_link7, child panda_link8, origin xyz=0 0 0.107 rpy=0 0 0
- added joint joint_world: type fixed, parent world, child panda_link0, origin xyz=0 0 0 rpy=0 0 0

Commit message: Gather some results with rosbag

File: urdf/container.xacro (robot description, xacro)
@@ -1,4 +1,46 @@
 <?xml version="1.0"?>
 <robot xmlns:xacro="http://www.ros.org/wiki/xacro" name="container">
+  <xacro:property name="mesh_scale" value="0.003 0.003 0.002"/>
+  <xacro:property name="mesh_origin_xyz" value="0 -0.027 0"/>
+  <xacro:property name="mesh_origin_rpy" value="-1.5708 0 0"/>
+  <link name="container_link">
+    <visual>
+      <origin xyz="${mesh_origin_xyz}" rpy="${mesh_origin_rpy}"/>
+      <geometry>
+        <mesh filename="package://vision_processing/urdf/Other_container.stl" scale="${mesh_scale}"/>
+      </geometry>
+      <material name="container_material">
+        <color rgba="1.0 1.0 1.0 1.0"/>
+      </material>
+    </visual>
+    <collision>
+      <origin xyz="${mesh_origin_xyz}" rpy="${mesh_origin_rpy}"/>
+      <geometry>
+        <mesh filename="package://vision_processing/urdf/Other_container_collision.stl" scale="${mesh_scale}"/>
+      </geometry>
+    </collision>
+    <inertial>
+      <mass value="0.3"/>
+      <inertia ixx="1e-3" ixy="0" ixz="0" iyy="1e-3" iyz="0" izz="1e-3"/>
+    </inertial>
+  </link>
+  <gazebo reference="container_link">
+    <material>Gazebo/White</material>
+  </gazebo>
+  <gazebo>
+    <static>true</static>
+    <plugin name="p3d_base_controller" filename="libgazebo_ros_p3d.so">
+      <alwaysOn>true</alwaysOn>
+      <updateRate>50.0</updateRate>
+      <bodyName>container_link</bodyName>
+      <topicName>container_pose</topicName>
+      <gaussianNoise>0.0</gaussianNoise>
+      <frameName>world</frameName>
+      <xyzOffsets>0 0 0</xyzOffsets>
+      <rpyOffsets>0 0 0</rpyOffsets>
+    </plugin>
+  </gazebo>
+</robot>
+<!--robot xmlns:xacro="http://www.ros.org/wiki/xacro" name="container">
   <xacro:property name="mesh_scale" value="0.025 0.025 0.025"/>
   <link name="container_link">
@@ -39,3 +81,3 @@
     </plugin>
   </gazebo>
-</robot>
+</robot-->

Commit message: Update

File: urdf/container.xacro (robot description, xacro)
@@ -82,2 +82,44 @@
   </gazebo>
 </robot-->
+<!--robot xmlns:xacro="http://www.ros.org/wiki/xacro" name="container">
+  <xacro:property name="mesh_scale" value="1 1 1"/>
+  <xacro:property name="mesh_origin_xyz" value="0 -0.027 0"/>
+  <xacro:property name="mesh_origin_rpy" value="-1.5708 0 0"/>
+  <link name="container_link">
+    <visual>
+      <origin xyz="${mesh_origin_xyz}" rpy="${mesh_origin_rpy}"/>
+      <geometry>
+        <mesh filename="package://vision_processing/urdf/urdf/simple_fish_bowl.glb" scale="${mesh_scale}"/>
+      </geometry>
+      <material name="container_material">
+        <color rgba="1.0 1.0 1.0 1.0"/>
+      </material>
+    </visual>
+    <collision>
+      <origin xyz="${mesh_origin_xyz}" rpy="${mesh_origin_rpy}"/>
+      <geometry>
+        <mesh filename="package://vision_processing/urdf/urdf/simple_fish_bowl.glb" scale="${mesh_scale}"/>
+      </geometry>
+    </collision>
+    <inertial>
+      <mass value="0.3"/>
+      <inertia ixx="1e-3" ixy="0" ixz="0" iyy="1e-3" iyz="0" izz="1e-3"/>
+    </inertial>
+  </link>
+  <gazebo reference="container_link">
+    <material>Gazebo/White</material>
+  </gazebo>
+  <gazebo>
+    <static>true</static>
+    <plugin name="p3d_base_controller" filename="libgazebo_ros_p3d.so">
+      <alwaysOn>true</alwaysOn>
+      <updateRate>50.0</updateRate>
+      <bodyName>container_link</bodyName>
+      <topicName>container_pose</topicName>
+      <gaussianNoise>0.0</gaussianNoise>
+      <frameName>world</frameName>
+      <xyzOffsets>0 0 0</xyzOffsets>
+      <rpyOffsets>0 0 0</rpyOffsets>
+    </plugin>
+  </gazebo>
+</robot-->
